File: V2/ECU_proj/DRV8262.kicad_sch (KiCad schematic)
At the start: 19 parts, among them IC1 DRV8262DDWR, J1 OUT1, J2 OUT2, J3 OUT4, J4 OUT3, J6 PGND

Commit message: Alpha Release
Parts:
- added C24: 1uF 100V, Capacitor_SMD:C_0402_1005Metric, symbol Device:C
- added C25: 100nF 100V, Capacitor_SMD:C_0402_1005Metric, symbol Device:C
Connections:
- net +3.3V: now also IC1.29 (MODE2), R7.1, C25.2
- net GND: now also C24.1, C25.1
- net VM: now also C24.2
- net at C23.1, IC1.24 (DVDD): no longer IC1.29 (MODE2), R7.1
