File: V2/ECU_proj/ECU_proj.kicad_pcb (KiCad board)
At the start: 2 copper layers, 91 x 35 mm, 48 parts, among them IC1 DRV8262DDWR, IC2 TC4421AVOA, IC3 TC4422AVOA, J1 OUT1, J10 Conn_02x03_Odd_Even, J11 Conn_01x01, J2 OUT2, J3 OUT4, J4 OUT3, J5 GND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

Commit message: Review before PCB production
Parts:
- added D2: LED, LED_SMD:LED_0402_1005Metric, F.Cu at (147.0, 72.5)
- added G***: LOGO, LOGO, F.Cu at (185.9, 79.3)
- moved C1 0.40 mm to (117.0, 72.5)
Routing:
- net +3.3V: track 73.4 -> 60.4 mm
- net /DRV8262/fault: track 47.6 -> 55.9 mm
- net Net-(IC1-VCP): track 3.83 -> 7.37 mm
- net /Attiny/trg1: track 18.4 -> 20.7 mm
- net GND: track 172.7 -> 170.4 mm, vias 111 -> 112
- net /Attiny/sens1: track 16.1 -> 18.2 mm
- net Net-(IC1-DVDD): track 17.3 -> 17.9 mm

Commit message: Alpha Release
Parts:
- added C24: 1uF 100V, Capacitor_SMD:C_0402_1005Metric, F.Cu at (120.0, 55.8)
- added C25: 100nF 100V, Capacitor_SMD:C_0402_1005Metric, F.Cu at (133.0, 81.4)
- moved R7 0.28 mm to (132.2, 77.6)
Connections:
- IC1 pad 29: Net-(IC1-DVDD) -> +3.3V
- R7 pad 1: Net-(IC1-DVDD) -> +3.3V
Routing:
- net GND: track 170.4 -> 188.2 mm, vias 112 -> 135
- net +3.3V: track 60.4 -> 74.0 mm, vias 0 -> 3
- net Net-(IC1-DVDD): track 17.9 -> 4.75 mm, vias 2 -> 0
- net /DRV8262/VM: track 46.9 -> 51.4 mm
- net /DRV8262/fault: track 55.9 -> 57.8 mm
- net /Mosfets/A1_12V: track 13.9 -> 15.6 mm
Other:
- board text added: "SDA ENABLE SCL FAULT TRG2 TRG1"
